File: saucey.kicad_sch (KiCad schematic)
At the start: 48 parts, among them J1 Conn_01x02_Socket, J2 USB_C_Receptacle_USB2.0_16P, M1 Motor_DC, M2 Motor_DC, M3 Motor_DC, M4 Motor_DC, Q1 AO3401A, Q3 SI2306, Q4 SI2306, Q5 SI2306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

Commit message: Add files via upload
Other:
- note added: "Half Bridge driving MOSFETs"
- note added: "Inertial Measurement Unit"
- note added: "Microcontroller"
- note added: "USB-C and Power"
- moved on the sheet: C10, C11, C12, C13, D1, D2, D3, D4, M1, M2, M3, M4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
